Commit message: Agrega configuración de URDF, Launch file y parámetros de SLAM para tetrabot en Ignition Fortress

File: urdf/gazebo/gazebo_plugins.xacro (robot description, xacro)
@@ -41,5 +41,5 @@
 <!-- =========== Lidar Sensor ============ -->
     <gazebo reference="lidar_link">
-        <sensor name='gpu_lidar' type='gpu_lidar'>"
+        <sensor name='gpu_lidar' type='gpu_lidar'>
             <pose relative_to='lidar_link'>0 0 0 0 0 0</pose>
             <topic>scan</topic>
@@ -134,108 +134,3 @@
   </light>
 </gazebo>
-<gazebo reference="faro_trasero_link">
-    <visual>
-      <material>
-        <ambient>1 0 0 1</ambient>
-        <diffuse>1 0 0 1</diffuse>
-        <specular>1 1 1 1</specular>
-        <emissive>1 0 0 1</emissive> </material>
-    </visual>
-    <light name="faro_trasero_luz" type="spot">
-      <pose>0 0 0 0 0 0</pose>
-      <diffuse>1 0 0 1</diffuse> <specular>.1 .1 .1 1</specular>
-      <attenuation>
-        <range>10</range>
-        <constant>0.5</constant>
-        <linear>0.01</linear>
-        <quadratic>0.001</quadratic>
-      </attenuation>
-      <direction>-1 0 0</direction>
-      <spot>
-        <inner_angle>0.1</inner_angle>
-        <outer_angle>0.5</outer_angle>
-        <falloff>1.2</falloff>
-      </spot>
-      <cast_shadows>true</cast_shadows>
-    </light>
-  </gazebo>
-<!-- CONFIGURACIÓN GAZEBO PARA SENSORES ULTRASÓNICOS -->
- <gazebo reference="ultrasonico_dere_link">
-    <sensor type="gpu_lidar" name="ultrasonico_der">
-      <pose>0 0 0 0 0 0</pose>
-      <visualize>true</visualize>
-      <update_rate>10</update_rate>
-      <topic>/ultrasonico/der</topic>
-      <ignition_frame_id>tetrabot/ultrasonico_dere_link</ignition_frame_id>
-      <ray>
-        <scan>
-          <horizontal>
-            <samples>5</samples>
-            <resolution>1</resolution>
-            <min_angle>-0.13</min_angle>
-            <max_angle>0.13</max_angle>
-          </horizontal>
-          <vertical>
-            <samples>5</samples>
-            <resolution>1</resolution>
-            <min_angle>-0.01</min_angle>
-            <max_angle>0.01</max_angle>
-          </vertical>
-        </scan>
-        <range>
-          <min>0.02</min>
-          <max>4.0</max>
-          <resolution>0.01</resolution>
-        </range>
-      </ray>
-    </sensor>
-  </gazebo>
-  <gazebo reference="ultrasonico_iz_link">
-    <sensor type="gpu_lidar" name="ultrasonico_iz">
-      <pose>0 0 0 0 0 0</pose>
-      <visualize>true</visualize>
-      <update_rate>10</update_rate>
-      <topic>/ultrasonico/iz</topic>
-      <ignition_frame_id>tetrabot/ultrasonico_iz_link</ignition_frame_id>
-      <ray>
-        <scan>
-          <horizontal>
-            <samples>5</samples>
-            <resolution>1</resolution>
-            <min_angle>-0.13</min_angle>
-            <max_angle>0.13</max_angle>
-          </horizontal>
-        </scan>
-        <range>
-          <min>0.02</min>
-          <max>4.0</max>
-          <resolution>0.01</resolution>
-        </range>
-      </ray>
-    </sensor>
-  </gazebo>
-  <gazebo reference="ultrasonico_tra_link">
-    <sensor type="gpu_lidar" name="ultrasonico_tra">
-      <pose>0 0 0 0 0 0</pose>
-      <visualize>true</visualize>
-      <update_rate>10</update_rate>
-      <topic>/ultrasonico/tra</topic>
-      <ignition_frame_id>tetrabot/ultrasonico_tra_link</ignition_frame_id>
-      <ray>
-        <scan>
-          <horizontal>
-            <samples>5</samples>
-            <resolution>1</resolution>
-            <min_angle>-0.13</min_angle>
-            <max_angle>0.13</max_angle>
-          </horizontal>
-        </scan>
-        <range>
-          <min>0.02</min>
-          <max>4.0</max>
-          <resolution>0.01</resolution>
-        </range>
-      </ray>
-    </sensor>
-  </gazebo>
 </robot>

File: urdf/modules/base_y_llantas.xacro (robot description, xacro)
@@ -3,5 +3,5 @@
 <!-- Onshape document_id: 3023829f8e4e5c564f6b4985 -->
 <robot xmlns:xacro="http://www.ros.org/wiki/xacro">
-  <!-- Link base footprint -->
+   <!-- Link base footprint -->
   <link name="base_footprint"/>
   <!-- Joint base footprint -->

File: urdf/modules/camara.xacro (robot description, xacro)
@@ -1,16 +1,20 @@
 <?xml version="1.0" ?>
+<!-- Generated using onshape-to-robot -->
+<!-- Onshape document_id: 3023829f8e4e5c564f6b4985 -->
 <robot xmlns:xacro="http://www.ros.org/wiki/xacro">
+<!-- Link camara_link -->
   <link name="camara_link">
     <inertial>
-      <origin xyz="-0 0 -0.00516528" rpy="0 0 0"/>
-      <mass value="0.0399941"/>
-      <inertia ixx="6.59521e-06" ixy="0" ixz="0" iyy="6.59521e-06" iyz="0" izz="1.04207e-05"/>
+      <origin xyz="3.9793e-08 -2.2226e-08 -0.00553286" rpy="0 0 0"/>
+      <mass value="0.0293384"/>
+      <inertia ixx="5.36338e-06" ixy="1.1e-11" ixz="-4e-12" iyy="5.36338e-06" iyz="4e-12" izz="8.08857e-06"/>
     </inertial>
+    <!-- Part camara_link -->
     <visual>
       <origin xyz="0 0 0.005" rpy="3.14159 -0 1.5708"/>
       <geometry>
-        <mesh filename="package://my_robot_description/assets/camara_t_s.stl"/>
+        <mesh filename="package://my_robot_description/assets/camara_link.stl"/>
       </geometry>
-      <material name="camara_t_s_material">
+      <material name="camara_link_material">
         <color rgba="0.262745 0.282353 0.301961 1"/>
       </material>
@@ -19,9 +23,10 @@
       <origin xyz="0 0 0.005" rpy="3.14159 -0 1.5708"/>
       <geometry>
-        <mesh filename="package://my_robot_description/assets/camara_t_s.stl"/>
+        <mesh filename="package://my_robot_description/assets/camara_link.stl"/>
       </geometry>
     </collision>
   </link>
-  <joint name="camara" type="fixed">
+  <!-- Joint from base_link to camara_link -->
+  <joint name="camara_joint" type="fixed">
     <origin xyz="0.115 0 0.135" rpy="0 0 0"/>
     <parent link="base_link"/>
@@ -30,30 +35,17 @@
     <limit effort="100" velocity="100"/>
   </joint>
+  <!--THIS IS A FIX TO CHANGE THE ORIENTATION SO IT WORKS WITH OPENCV (ALWAYS INCLUDE)
+  generate an optical frame
+  http://www.ros.org/reps/rep-0103.html#suffix-frames
+  so that ros and opencv can operate on the camera frame correctly -->
   <link name="camera_optical_link">
   </link>
   <joint name="camera_optical_joint" type="fixed">
+      <!-- these values have to be these values otherwise the gazebo camera
+          image won't be aligned properly with the frame it is supposedly
+          originating from -->
       <origin xyz="0 0 0" rpy="${-pi/2} 0 ${-pi/2}"/>
       <parent link="camara_link"/>
       <child link="camera_optical_link"/>
   </joint>
-  <gazebo reference="camara_link">
-    <sensor name="depth_camera" type="rgbd_camera">
-      <always_on>true</always_on>
-      <update_rate>20.0</update_rate>
-      <topic>camera</topic>
-      <camera>
-        <horizontal_fov>1.047198</horizontal_fov>
-        <image>
-          <width>640</width>
-          <height>480</height>
-          <format>RGB_INT8</format>
-        </image>
-        <clip>
-          <near>0.05</near>
-          <far>8.0</far>
-        </clip>
-        <optical_frame_id>camera_optical_link</optical_frame_id>
-      </camera>
-    </sensor>
-  </gazebo>
 </robot>

File: urdf/modules/lidar.xacro (robot description, xacro)
@@ -3,5 +3,5 @@
 <!-- Onshape document_id: 3023829f8e4e5c564f6b4985 -->
 <robot xmlns:xacro="http://www.ros.org/wiki/xacro">
-<!-- Link lidar_link -->
+  <!-- Link lidar_link -->
   <link name="lidar_link">
     <inertial>

File: urdf/robot.urdf (robot description, URDF)
Before this commit: robot None, 9 links, 9 joints
Links:
- removed link ultrasonico_der_dia_link
- removed link ultrasonico_dere_link
- removed link ultrasonico_iz_dia_link
- removed link ultrasonico_iz_link
- removed link ultrasonico_tra_link
- added link base_link, mass 16.1488; collision mesh filename=package://my_robot_description/assets/base_link.stl; visual mesh filename=package://my_robot_description/assets/base_link.stl
- added link camara_link, mass 0.0293384; collision mesh filename=package://my_robot_description/assets/camara_link.stl; visual mesh filename=package://my_robot_description/assets/camara_link.stl
- added link lidar_link, mass 0.0591873; collision mesh filename=package://my_robot_description/assets/lidar_link.stl; visual mesh filename=package://my_robot_description/assets/lidar_link.stl
- added link llanta_dere_del, mass 0.324568; collision mesh filename=package://my_robot_description/assets/llanta_dere_del.stl; visual mesh filename=package://my_robot_description/assets/llanta_dere_del.stl
- added link llanta_dere_tra, mass 0.324568; collision mesh filename=package://my_robot_description/assets/llanta_dere_tra.stl; visual mesh filename=package://my_robot_description/assets/llanta_dere_tra.stl
- added link llanta_iz_del, mass 0.324568; collision mesh filename=package://my_robot_description/assets/llanta_iz_del.stl; visual mesh filename=package://my_robot_description/assets/llanta_iz_del.stl
- added link llanta_iz_tra, mass 0.324568; collision mesh filename=package://my_robot_description/assets/llanta_iz_tra.stl; visual mesh filename=package://my_robot_description/assets/llanta_iz_tra.stl
- added link ultra_t, mass 0.00553386; collision mesh filename=package://my_robot_description/assets/ultra_t.stl; visual mesh filename=package://my_robot_description/assets/ultra_t.stl
- added link ultra_t_2, mass 0.00553386; collision mesh filename=package://my_robot_description/assets/ultra_t.stl; visual mesh filename=package://my_robot_description/assets/ultra_t.stl
- added link ultra_t_3, mass 0.00553386; collision mesh filename=package://my_robot_description/assets/ultra_t.stl; visual mesh filename=package://my_robot_description/assets/ultra_t.stl
- added link ultra_t_4, mass 0.00553386; collision mesh filename=package://my_robot_description/assets/ultra_t.stl; visual mesh filename=package://my_robot_description/assets/ultra_t.stl
- added link ultra_t_5, mass 0.00553386; collision mesh filename=package://my_robot_description/assets/ultra_t.stl; visual mesh filename=package://my_robot_description/assets/ultra_t.stl
Joints:
- removed joint antena_joint
- removed joint faro_delantero_joint
- removed joint faro_trasero_joint
- removed joint tapa_joint
- removed joint ultrasonico_der_dia_joint
- removed joint ultrasonico_dere_joint
- removed joint ultrasonico_iz_dia_joint
- removed joint ultrasonico_iz_joint
- removed joint ultrasonico_tra_joint
- added joint antena: type fixed, parent base_link, child antena_link, origin xyz=-0.12 -0.09 0.1125 rpy=3.14159 -0 0, axis 0 0 1, limit effort=100 velocity=100
- added joint camara: type fixed, parent base_link, child camara_link, origin xyz=0.115 0 0.135 rpy=-1.5708 -0 1.5708, axis 0 0 1, limit effort=100 velocity=100
- added joint faro_delantero: type fixed, parent base_link, child faro_delantero_link, origin xyz=0.12 0 0.06 rpy=-1.5708 -0 1.5708, axis 0 0 1, limit effort=100 velocity=100
- added joint faro_trasero: type fixed, parent base_link, child faro_trasero_link, origin xyz=-0.12 -0 0.1125 rpy=3.14159 -0 0, axis 0 0 1, limit effort=100 velocity=100
- added joint lidar: type fixed, parent base_link, child lidar_link, origin xyz=0.08 0 0.18 rpy=3.14159 -0 0, axis 0 0 1, limit effort=100 velocity=100
- added joint llanta_dere_del: type revolute, parent base_link, child llanta_dere_del, origin xyz=0.0441 -0.095 0.0162 rpy=-1.5708 -0 0, axis 0 0 1, limit lower=-3.141592653589793 upper=3.141592653589793 effort=100 velocity=100
- added joint llanta_dere_tra: type revolute, parent base_link, child llanta_dere_tra, origin xyz=-0.0859 -0.095 0.0162 rpy=-1.5708 -0 0, axis 0 0 1, limit lower=-3.141592653589793 upper=3.141592653589793 effort=100 velocity=100
- added joint llanta_iz_del: type revolute, parent base_link, child llanta_iz_del, origin xyz=0.0441 0.095 0.0162 rpy=1.5708 -0 0, axis 0 0 1, limit lower=-3.141592653589793 upper=3.141592653589793 effort=100 velocity=100
- added joint llanta_iz_tra: type revolute, parent base_link, child llanta_iz_tra, origin xyz=-0.0859 0.095 0.0162 rpy=1.5708 -0 0, axis 0 0 1, limit lower=-3.141592653589793 upper=3.141592653589793 effort=100 velocity=100
- added joint tapa: type fixed, parent base_link, child tapa_link, origin xyz=-0.1 0.09 0.16 rpy=3.14159 -0 0, axis 0 0 1, limit effort=100 velocity=100
- added joint ultrasonico_der_dia: type fixed, parent base_link, child ultra_t_2, origin xyz=0.0901178 -0.0801178 0.085 rpy=-1.5708 -0 0.785398, axis 0 0 1, limit effort=100 velocity=100
- added joint ultrasonico_dere: type fixed, parent base_link, child ultra_t, origin xyz=0 -0.1025 0.085 rpy=-1.5708 -0 0, axis 0 0 1, limit effort=100 velocity=100
- added joint ultrasonico_iz: type fixed, parent base_link, child ultra_t_4, origin xyz=-0 0.1025 0.085 rpy=1.5708 -0 0, axis 0 0 1, limit effort=100 velocity=100
- added joint ultrasonico_iz_dia: type fixed, parent base_link, child ultra_t_3, origin xyz=0.0901178 0.0801178 0.085 rpy=1.5708 -0 -0.785398, axis 0 0 1, limit effort=100 velocity=100
- added joint ultrasonico_tra: type fixed, parent base_link, child ultra_t_5, origin xyz=-0.1125 0 0.04125 rpy=1.5708 -0 1.5708, axis 0 0 1, limit effort=100 velocity=100
