Commit message: Actualización: Integración de servidor web Flask, control de Nav2 y motor

File: urdf/modules/lidar.xacro (robot description, xacro)
@@ -29,5 +29,5 @@
   <!-- Joint from base_link to lidar_link -->
   <joint name="lidar_joint" type="fixed">
-    <origin xyz="0.08 0 0.18" rpy="0 0 0"/>
+    <origin xyz="0.08 0 0.19" rpy="0 0 0"/>
     <parent link="base_link"/>
     <child link="lidar_link"/>
